Commit message: move reach_env to tasks, add gripper functions

File: ur5_gym/models/ur5/ur5_gripper.urdf (robot description, URDF)
Before this commit: robot ur5, 11 links, 10 joints
Links:
- added link left_inner_finger, mass 0.0104003125914103; collision mesh filename=robotiq_2f_85_gripper_visualization/meshes/collision/roboti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 scale=0.001 0.001 0.001; visual mesh filename=robotiq_2f_85_gripper_visualization/meshes/visual/robotiq_a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 scale=0.001 0.001 0.001
- added link left_inner_finger_pad, mass 1; collision box size=0.022 0.00635 0.0375; visual box size=0.022 0.00635 0.0375
- added link left_inner_knuckle, mass 0.0271177346495152; collision mesh filename=robotiq_2f_85_gripper_visualization/meshes/collision/roboti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 scale=0.001 0.001 0.001; visual mesh filename=robotiq_2f_85_gripper_visualization/meshes/visual/robotiq_a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 scale=0.001 0.001 0.001
- added link left_outer_finger, mass 0.022614240507152; collision mesh filename=robotiq_2f_85_gripper_visualization/meshes/collision/roboti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 scale=0.001 0.001 0.001; visual mesh filename=robotiq_2f_85_gripper_visualization/meshes/visual/robotiq_a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 scale=0.001 0.001 0.001
- added link left_outer_knuckle, mass 0.00853198276973456; collision mesh filename=robotiq_2f_85_gripper_visualization/meshes/collision/roboti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 scale=0.001 0.001 0.001; visual mesh filename=robotiq_2f_85_gripper_visualization/meshes/visual/robotiq_a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 scale=0.001 0.001 0.001
- added link right_inner_finger, mass 0.0104003125914103; collision mesh filename=robotiq_2f_85_gripper_visualization/meshes/collision/roboti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 scale=0.001 0.001 0.001; visual mesh filename=robotiq_2f_85_gripper_visualization/meshes/visual/robotiq_a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 scale=0.001 0.001 0.001
- added link right_inner_finger_pad, mass 1; collision box size=0.022 0.00635 0.0375; visual box size=0.022 0.00635 0.0375
- added link right_inner_knuckle, mass 0.0271177346495152; collision mesh filename=robotiq_2f_85_gripper_visualization/meshes/collision/roboti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 scale=0.001 0.001 0.001; visual mesh filename=robotiq_2f_85_gripper_visualization/meshes/visual/robotiq_a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 scale=0.001 0.001 0.001
- added link right_outer_finger, mass 0.022614240507152; collision mesh filename=robotiq_2f_85_gripper_visualization/meshes/collision/roboti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 scale=0.001 0.001 0.001; visual mesh filename=robotiq_2f_85_gripper_visualization/meshes/visual/robotiq_a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 scale=0.001 0.001 0.001
- added link right_outer_knuckle, mass 0.00853198276973456; collision mesh filename=robotiq_2f_85_gripper_visualization/meshes/collision/roboti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 scale=0.001 0.001 0.001; visual mesh filename=robotiq_2f_85_gripper_visualization/meshes/visual/robotiq_a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 scale=0.001 0.001 0.001
- added link robotiq_arg2f_base_link, mass 0.22652; collision mesh filename=robotiq_2f_85_gripper_visualization/meshes/collision/roboti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; visual mesh filename=robotiq_2f_85_gripper_visualization/meshes/visual/robotiq_a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 scale=0.001 0.001 0.001
- added link tool0_ee
- link tool0: mass None -> 0; geometry visual cylinder length=0.14 radius=0.01
Joints:
- added joint hand_to_grip: type fixed, parent tool0, child robotiq_arg2f_base_link, origin xyz=0.0 0.0 0.0 rpy=0 0.0 0.0
- added joint left_inner_finger_joint: type revolute, parent left_outer_finger, child left_inner_finger, origin xyz=0 0.0061 0.0471 rpy=0 0 0, axis 1 0 0, limit lower=0 upper=0.8757 effort=1000 velocity=2.0, mimic joint=left_outer_knuckle_joint multiplier=-1 offset=0
- added joint left_inner_finger_pad_joint: type fixed, parent left_inner_finger, child left_inner_finger_pad, origin xyz=0 -0.0220203446692936 0.03242 rpy=0 0 0, axis 0 0 1
- added joint left_inner_knuckle_joint: type revolute, parent robotiq_arg2f_base_link, child left_inner_knuckle, origin xyz=0 -0.0127 0.06142 rpy=0 0 3.141592653589793, axis 1 0 0, limit lower=0 upper=0.8757 effort=1000 velocity=2.0, mimic joint=left_outer_knuckle_joint multiplier=1 offset=0
- added joint left_outer_finger_joint: type fixed, parent left_outer_knuckle, child left_outer_finger, origin xyz=0 0.0315 -0.0041 rpy=0 0 0, axis 1 0 0
- added joint left_outer_knuckle_joint: type revolute, parent robotiq_arg2f_base_link, child left_outer_knuckle, origin xyz=0 -0.0306011 0.054904 rpy=0 0 3.141592653589793, axis 1 0 0, limit lower=0 upper=0.8 effort=1000 velocity=2.0
- added joint right_inner_finger_joint: type revolute, parent right_outer_finger, child right_inner_finger, origin xyz=0 0.0061 0.0471 rpy=0 0 0, axis 1 0 0, limit lower=0 upper=0.8757 effort=1000 velocity=2.0, mimic joint=left_outer_knuckle_joint multiplier=-1 offset=0
- added joint right_inner_finger_pad_joint: type fixed, parent right_inner_finger, child right_inner_finger_pad, origin xyz=0 -0.0220203446692936 0.03242 rpy=0 0 0, axis 0 0 1
- added joint right_inner_knuckle_joint: type revolute, parent robotiq_arg2f_base_link, child right_inner_knuckle, origin xyz=0 0.0127 0.06142 rpy=0 0 0.0, axis 1 0 0, limit lower=0 upper=0.8757 effort=1000 velocity=2.0, mimic joint=left_outer_knuckle_joint multiplier=1 offset=0
- added joint right_outer_finger_joint: type fixed, parent right_outer_knuckle, child right_outer_finger, origin xyz=0 0.0315 -0.0041 rpy=0 0 0, axis 1 0 0
- added joint right_outer_knuckle_joint: type revolute, parent robotiq_arg2f_base_link, child right_outer_knuckle, origin xyz=0 0.0306011 0.054904 rpy=0 0 0, axis 1 0 0, limit lower=0 upper=0.81 effort=1000 velocity=2.0, mimic joint=left_outer_knuckle_joint multiplier=1 offset=0
- added joint wrist_3_link-tool0_ee_fixed_joint: type fixed, parent tool0, child tool0_ee, origin xyz=0 0 0.15 rpy=0 0 0
